File: kicad controller/controller.kicad_pcb (KiCad board)
At the start: 2 copper layers, 51 parts, among them P1 CONN_4_V, P2 CONN_02X05, P3 CONN_01X01, P4 CONN_01X01, P5 CONN_01X01, Q1 MOS_N, Q2 MOS_N, Q3 MOS_N, Q4 MOS_N, Q5 MOS_N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

Commit message: updated pcd
Routing:
- net /A: track 11.0 -> 60.2 mm, vias 0 -> 2
- net /B: track 45.7 -> 65.6 mm, vias 2 -> 3
- net /C: track 25.6 -> 45.0 mm, vias 1 -> 2
- net VPP: track 70.3 -> 67.1 mm, vias 3 -> 0
- net /BLS: track 2.77 -> 5.31 mm
- net /ALS: track 2.41 -> 4.95 mm
- net /CLS: track 2.77 -> 5.31 mm
- net /GAH: track 9.35 -> 10.3 mm
