File: kicad controller/controller.sch (KiCad schematic (older format))
At the start: 53 parts, among them P1 CONN_4_V, P2 CONN_02X05, P3 CONN_01X01, P4 CONN_01X01, P5 CONN_01X01, Q1 MOS_N, Q2 MOS_N, Q3 MOS_N, Q4 MOS_N, Q5 MOS_N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

Commit message: grml
Parts:
- added C10, C11, C12, C13, C7, C9: 100n, SMD_Packages:SMD-0603_r, symbol C
- added C8: 47u, SMD_Packages:SMD-0603_r, symbol C
- D2, D3, D5, D6, D8, D9: footprint SMD_Packages:SMD-0603_r -> SMD_Packages:DO-214-AC_SMA
Connections:
- net +12V: now also C7.1 (A), C8.1 (A)
- net +5V: now also C10.1 (A), C11.1 (A), C12.1 (A), C9.1 (A)
- net +5VA: now also C13.1 (A)
- net DGND: now also C10.2 (B), C11.2 (B), C12.2 (B), C9.2 (B)
- net GND: now also C13.2 (B), C7.2 (B), C8.2 (B)
- net BOOTB: now reaches C2.1 (A), D4.2 (K), U2.1 (BHB)
- net BOOTC: now reaches C3.1 (A), D7.2 (K), U2.13 (CHB)
- net BOOTA: now reaches C1.1 (A), D1.2 (K), U2.16 (AHB)
