File: kicad controller/_autosave-controller.kicad_pcb (KiCad board)
At the start: 2 copper layers, 56 x 56 mm, 62 parts, among them P1 CONN_4_V, P2 CONN_02X05, P3 CONN_01X01, P4 CONN_01X01, P5 CONN_01X01, Q1 MOS_N, Q2 MOS_N, Q3 MOS_N, Q4 MOS_N, Q5 MOS_N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

Commit message: added thermals to mosfets
Routing:
- net /A: track 53.5 -> 45.6 mm, vias 3 -> 2
- net /B: track 57.8 -> 55.2 mm, vias 3 -> 2
- net /C: track 37.6 -> 35.1 mm, vias 3 -> 2
Changed lines of the file:
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@@
     (thickness 1.6)
     (drawings 8)
-    (tracks 425)
+    (tracks 422)
     (zones 0)
     (modules 62)
@@
   )
   (setup
-    (last_trace_width 0.254)
+    (last_trace_width 0.6)
     (user_trace_width 0.254)
     (user_trace_width 0.6)
@@
   (segment (start 173.863 68.06692) (end 176.40808 70.612) (width 0.6) (layer B.Cu) (net 2))
   (segment (start 173.863 67.68592) (end 173.863 68.06692) (width 0.6) (layer B.Cu) (net 2))
+  (segment (start 187.833 68.834) (end 187.833 71.628) (width 0.6) (layer B.Cu) (net 3))
+  (segment (start 197.594001 73.305001) (end 199.136 71.763002) (width 0.6) (layer B.Cu) (net 3))
+  (segment (start 187.833 71.628) (end 189.510001 73.305001) (width 0.6) (layer B.Cu) (net 3))
+  (segment (start 189.510001 73.305001) (end 197.594001 73.305001) (width 0.6) (layer B.Cu) (net 3))
+  (segment (start 199.136 71.763002) (end 199.136 67.294) (width 0.6) (layer B.Cu) (net 3))
+  (segment (start 199.136 67.294) (end 203.15 63.28) (width 0.6) (layer B.Cu) (net 3))
+  (segment (start 203.15 63.28) (end 203.25 63.28) (width 0.6) (layer B.Cu) (net 3))
   (segment (start 208.095 60.325) (end 206.27 60.325) (width 0.254) (layer F.Cu) (net 3))
   (segment (start 206.27 60.325) (end 205.95 60.005) (width 0.254) (layer F.Cu) (net 3))
@@
   (segment (start 182.753 69.85) (end 183.388 69.215) (width 0.6) (layer B.Cu) (net 3))
   (segment (start 182.118 69.85) (end 182.753 69.85) (width 0.6) (layer B.Cu) (net 3))
-  (segment (start 189.510001 73.305001) (end 197.458999 73.305001) (width 0.6) (layer B.Cu) (net 3))
-  (segment (start 187.833 71.628) (end 189.510001 73.305001) (width 0.6) (layer B.Cu) (net 3))
-  (segment (start 187.833 68.834) (end 187.833 71.628) (width 0.6) (layer B.Cu) (net 3))
-  (segment (start 197.594001 73.305001) (end 199.136 71.763002) (width 0.6) (layer B.Cu) (net 3))
-  (segment (start 197.458999 73.305001) (end 197.594001 73.305001) (width 0.6) (layer B.Cu) (net 3))
   (segment (start 180.96992 69.85) (end 180.20792 70.612) (width 0.6) (layer B.Cu) (net 3))
   (segment (start 182.118 69.85) (end 180.96992 69.85) (width 0.6) (layer B.Cu) (net 3))
   (segment (start 205.867 58.293) (end 205.486 58.674) (width 0.6) (layer F.Cu) (net 3))
-  (via (at 204.724 58.674) (size 1) (drill 0.3) (layers F.Cu B.Cu) (net 3))
   (segment (start 205.486 58.674) (end 205.431106 58.674) (width 0.6) (layer F.Cu) (net 3))
   (segment (start 205.431106 58.674) (end 204.724 58.674) (width 0.6) (layer F.Cu) (net 3))
@@
   (segment (start 205.95 59.28) (end 205.344 58.674) (width 0.6) (layer F.Cu) (net 3))
   (segment (start 205.344 58.674) (end 204.724 58.674) (width 0.6) (layer F.Cu) (net 3))
-  (segment (start 200.025 58.674) (end 204.724 58.674) (width 0.6) (layer B.Cu) (net 3))
-  (segment (start 199.136 59.563) (end 200.025 58.674) (width 0.6) (layer B.Cu) (net 3))
-  (segment (start 199.136 71.763002) (end 199.136 59.563) (width 0.6) (layer B.Cu) (net 3))
   (segment (start 175.895 53.975) (end 175.895 55.626) (width 0.6) (layer F.Cu) (net 4))
   (segment (start 175.895 55.626) (end 175.641 55.88) (width 0.6) (layer F.Cu) (net 4))
@@
   (segment (start 175.641 55.88) (end 173.863 55.88) (width 0.6) (layer F.Cu) (net 4))
   (segment (start 179.451 59.69508) (end 179.451 57.77992) (width 0.6) (layer B.Cu) (net 5))
+  (segment (start 203.25 47.21) (end 201.5 47.21) (width 0.6) (layer B.Cu) (net 6))
+  (segment (start 201.5 47.21) (end 201.466 47.244) (width 0.6) (layer B.Cu) (net 6))
+  (segment (start 201.466 47.244) (end 199.644 47.244) (width 0.6) (layer B.Cu) (net 6))
   (segment (start 183.094552 64.760778) (end 183.094552 63.210448) (width 0.6) (layer F.Cu) (net 6))
   (segment (start 183.094552 63.210448) (end 183.44 62.865) (width 0.6) (layer F.Cu) (net 6))
@@
   (segment (start 204.851 44.704) (end 204.851 44.936) (width 0.254) (layer F.Cu) (net 6))
   (segment (start 204.851 44.936) (end 205.95 46.035) (width 0.254) (layer F.Cu) (net 6))
-  (via (at 204.851 44.704) (size 1) (drill 0.3) (layers F.Cu B.Cu) (net 6))
   (segment (start 204.4 48.26) (end 204.47 48.26) (width 2) (layer F.Cu) (net 6))
   (segment (start 181.828694 63.49492) (end 183.094552 64.760778) (width 0.6) (layer B.Cu) (net 6))
@@
   (segment (start 190.588999 49.091649) (end 190.588999 45.333999) (width 0.6) (layer F.Cu) (net 6))
   (segment (start 196.731001 46.744001) (end 197.231 47.244) (width 0.6) (layer F.Cu) (net 6))
-  (segment (start 202.184 44.704) (end 199.644 47.244) (width 0.6) (layer B.Cu) (net 6))
-  (segment (start 204.851 44.704) (end 202.184 44.704) (width 0.6) (layer B.Cu) (net 6))
   (segment (start 199.644 47.244) (end 197.231 47.244) (width 0.6) (layer B.Cu) (net 6))
   (segment (start 175.90008 74.295) (end 175.90008 75.50028) (width 0.6) (layer B.Cu) (net 7))
   (segment (start 175.90008 75.50028) (end 179.10008 78.70028) (width 0.6) (layer B.Cu) (net 7))
   (segment (start 179.10008 78.70028) (end 179.10008 79) (width 0.6) (layer B.Cu) (net 7))
+  (segment (start 203.25 75.15) (end 201.5 75.15) (width 0.6) (layer B.Cu) (net 8))
+  (segment (start 201.5 75.15) (end 200.958 75.692) (width 0.6) (layer B.Cu) (net 8))
+  (segment (start 200.958 75.692) (end 196.716617 75.692) (width 0.6) (layer B.Cu) (net 8))
+  (segment (start 196.716617 75.692) (end 196.088 75.692) (width 0.6) (layer B.Cu) (net 8))
   (segment (start 204.4 76.2) (end 205.95 74.65) (width 0.254) (layer F.Cu) (net 8))
   (segment (start 205.95 74.65) (end 205.95 73.975) (width 0.254) (layer F.Cu) (net 8))
@@
   (segment (start 204.4 76.2) (end 205.95 77.75) (width 0.254) (layer F.Cu) (net 8))
   (segment (start 205.95 77.75) (end 205.95 78.425) (width 0.254) (layer F.Cu) (net 8))
-  (via (at 204.724 72.771) (size 1) (drill 0.3) (layers F.Cu B.Cu) (net 8))
   (via (at 183.134 73.406) (size 0.8) (drill 0.4) (layers F.Cu B.Cu) (net 8))
   (segment (start 181.483 73.66) (end 182.88 73.66) (width 0.6) (layer B.Cu) (net 8))
@@
   (segment (start 193.421 73.025) (end 195.643501 75.247501) (width 0.6) (layer F.Cu) (net 8))
   (segment (start 195.643501 75.247501) (end 196.088 75.692) (width 0.6) (layer F.Cu) (net 8))
-  (segment (start 196.716617 75.692) (end 196.088 75.692) (width 0.6) (layer B.Cu) (net 8))
-  (segment (start 199.39 75.692) (end 196.716617 75.692) (width 0.6) (layer B.Cu) (net 8))
-  (segment (start 202.311 72.771) (end 199.39 75.692) (width 0.6) (layer B.Cu) (net 8))
-  (segment (start 204.724 72.771) (end 202.311 72.771) (width 0.6) (layer B.Cu) (net 8))
   (segment (start 204.746 72.771) (end 205.95 73.975) (width 0.6) (layer F.Cu) (net 8))
   (segment (start 204.724 72.771) (end 204.746 72.771) (width 0.6) (layer F.Cu) (net 8))
@@
     (polygon
       (pts
-        (xy 201.93 45.72) (xy 201.93 50.8) (xy 206.756 50.8) (xy 206.756 45.72)
+        (xy 201.93 45.72) (xy 201.93 50.8) (xy 206.883 50.8) (xy 206.883 45.72)
       )
     )
@@
     (polygon
       (pts
-        (xy 209.55 45.72) (xy 209.55 50.8) (xy 213.995 50.8) (xy 213.995 45.72)
+        (xy 209.55 45.72) (xy 209.55 50.8) (xy 214.503 50.8) (xy 214.503 45.72)
       )
     )
@@
     (polygon
       (pts
-        (xy 201.93 59.69) (xy 201.93 64.77) (xy 206.756 64.77) (xy 206.756 59.69)
+        (xy 201.93 59.69) (xy 201.93 64.77) (xy 206.883 64.77) (xy 206.883 59.69)
       )
     )
@@
     (polygon
       (pts
-        (xy 209.55 59.69) (xy 209.55 64.77) (xy 213.995 64.77) (xy 213.995 59.69)
+        (xy 209.55 59.69) (xy 209.55 64.77) (xy 214.503 64.77) (xy 214.503 59.69)
       )
     )
@@
     (polygon
       (pts
-        (xy 209.55 73.66) (xy 209.55 78.74) (xy 214.376 78.74) (xy 214.376 73.66)
+        (xy 209.55 73.66) (xy 209.55 78.74) (xy 214.503 78.74) (xy 214.503 73.66)
       )
     )
@@
     (polygon
       (pts
-        (xy 201.93 73.66) (xy 201.93 78.74) (xy 206.756 78.74) (xy 206.756 73.66)
+        (xy 201.93 73.66) (xy 201.93 78.74) (xy 206.883 78.74) (xy 206.883 73.66)
       )
     )
